File: HDC1080Breakout.kicad_pcb (KiCad board)
At the start: 2 copper layers, 10 x 10 mm, 8 parts, among them J1 Conn_01x04, U1 HDC1080

Commit message: Add files via upload
Parts:
- added G***: LOGO, LOGO, B.Cu at (2.50, 4.50)
